File: dualpress/dualpress.kicad_sch (KiCad schematic)
At the start: 19 parts, among them J1 WATCH_RELAIS, J2 CTRL_RELAIS, J3 WATCH_PRESSURE, J4 WATCH_VALVE, U1 ESP32-S3-DEVKITC-1-N8R2, U2 2.8" Touch Display SPI 14x1, U3 PC817, U5 AMS1117

Commit message: base layout done
Parts:
- removed C1, C4: 10u, Capacitor_Tantalum_SMD:CP_EIA-3528-21_Kemet-B_HandSolder, symbol Device:C_Polarized
- removed C2, C3: 1u, Capacitor_SMD:C_0805_2012Metric, symbol Device:C
- removed D1, D2: LED, Diode_SMD:D_0201_0603Metric, symbol Device:LED
- removed F1: Polyfuse, symbol Device:Polyfuse
- removed J1: WATCH_RELAIS, Connector_JST:JST_XH_B2B-XH-AM_1x02_P2.50mm_Vertical, symbol Connector:Screw_Terminal_01x02
- removed J2: CTRL_RELAIS, Connector_JST:JST_XH_B2B-XH-AM_1x02_P2.50mm_Vertical, symbol Connector:Conn_01x03_Socket
- removed J3: WATCH_PRESSURE, Connector_JST:JST_XH_B2B-XH-AM_1x02_P2.50mm_Vertical, symbol Connector:Conn_01x03_Socket
- removed J4: WATCH_VALVE, Connector_JST:JST_XH_B2B-XH-AM_1x02_P2.50mm_Vertical, symbol Connector:Conn_01x03_Socket
- removed JP1: Jumper_2_Open, Connector_PinHeader_2.54mm:PinHeader_1x02_P2.54mm_Vertical, symbol Jumper:Jumper_2_Open
- removed R1: 470, Resistor_SMD:R_0805_2012Metric, symbol Device:R
- removed R2: R, symbol Device:R
- removed R3: 1k, Resistor_SMD:R_0805_2012Metric, symbol Device:R
- removed U1: ESP32-S3-DEVKITC-1-N8R2, 01_dualpress:XCVR_ESP32-S3-DEVKITC-1-N8R2, symbol 01_dualpress:ESP32-S3-DEVKITC-1-N8R2
- removed U2: 2.8" Touch Display SPI 14x1, Connector_PinHeader_2.54mm:PinHeader_1x14_P2.54mm_Vertical, symbol 01_dualpress:2.8{dblquote} Touch Display SPI 14x1
- removed U3: PC817, Package_DIP:DIP-4_W7.62mm, symbol Isolator:PC817
- removed U5: AMS1117, PCM_JLCPCB:SOT-223-3_L6.5-W3.4-P2.30-LS7.0-BR, symbol PCM_JLCPCB-Power:LDO, 3.3V, 1A
- added C10: 1u, Capacitor_SMD:C_0805_2012Metric, symbol Device:C
- added C11: 100nF, PCM_JLCPCB:C_0603, symbol PCM_JLCPCB-Capacitors:0603,100nF
- added C9: 10uF, PCM_JLCPCB:C_0603, symbol PCM_JLCPCB-Capacitors:0603,10uF,(2)
- added R15: 0Ω, PCM_JLCPCB:R_0603, symbol PCM_JLCPCB-Resistors:0603,0Ω
- added R9: 10kΩ, PCM_JLCPCB:R_0603, symbol PCM_JLCPCB-Resistors:0603,10kΩ
- added U4: (no value), symbol 01_dualpress:ESP32-S2-WROOM-1-N16R8
Connections:
- net +3V3: now also C10.1, C11.1, C11.2, C9.1, C9.2, R15.2, U4.1 (GND)
- new net: U4.40 (GND), U4.41 (GND)
- new net CHIP_PU: C10.2, R9.1, U4.3 (EN)
- new net ESP_3V3: R15.1, R9.2, U4.2 (3V3)
- new net GPIO0: U4.27 (GPIO0/BOOT/STRAP)
- new net GPIO1: U4.39 (GPIO1)
- new net GPIO10: U4.18 (GPIO10)
- new net GPIO11: U4.19 (GPIO11)
- new net GPIO12: U4.20 (GPIO12)
- new net GPIO13: U4.21 (GPIO13)
- new net GPIO14: U4.22 (GPIO14)
- new net GPIO15: U4.8 (GPIO15)
- new net GPIO16: U4.9 (GPIO16)
- new net GPIO17: U4.10 (GPIO17)
- new net GPIO18: U4.11 (GPIO18)
- new net GPIO19: U4.13 (GPIO19/USB_D-)
- new net GPIO2: U4.38 (GPIO2)
- new net GPIO20: U4.14 (GPIO20/USB_D+)
- new net GPIO21: U4.23 (GPIO21)
- new net GPIO38: U4.31 (GPIO38)
- new net GPIO39: U4.32 (MTCK/GPIO39)
- new net GPIO4: U4.4 (GPIO4)
- new net GPIO40: U4.33 (MTDO/GPIO40)
- new net GPIO41: U4.34 (MTDI/GPIO41)
- new net GPIO42: U4.35 (MTMS/GPIO42)
- new net GPIO47: U4.24 (GPIO47)
- new net GPIO48: U4.25 (GPIO48)
- new net GPIO5: U4.5 (GPIO5)
- new net GPIO6: U4.6 (GPIO6)
- new net GPIO7: U4.7 (GPIO7)
- new net GPIO8: U4.12 (GPIO8)
- new net GPIO9: U4.17 (GPIO9)
- new net U0RXD: U4.36 (U0RXD/GPIO44)
- new net U0TXD: U4.37 (U0TXD/GPIO43)
- no-connect marks 0 -> 6
Other:
- added sheet DISPLAY (display.kicad_sch)
- added sheet PWR SUPPLY (pwr_supply.kicad_sch)
- added sheet SENSORS (sensors.kicad_sch)
- added sheet USB (untitled.kicad_sch)
- added sheet USB SERIAL (usb_serial.kicad_sch)
