File: dualpress/dualpress.kicad_sch (KiCad schematic)
At the start: 25 parts, among them Q2 SS8050, Q3 SS8050, U1 LD1117S33TR_SOT223

Commit message: before remove footprints
Parts:
- removed C10: 1u, Capacitor_SMD:C_0805_2012Metric, symbol Device:C
- removed C11: 100nF, PCM_JLCPCB:C_0603, symbol PCM_JLCPCB-Capacitors:0603,100nF
- removed C9: 10uF, PCM_JLCPCB:C_0603, symbol PCM_JLCPCB-Capacitors:0603,10uF,(2)
- removed R15: 0Ω, PCM_JLCPCB:R_0603, symbol PCM_JLCPCB-Resistors:0603,0Ω
- added C15: 10uF, PCM_JLCPCB:C_0805, symbol PCM_JLCPCB-Capacitors:0805,10uF
- added C6: 100nF, PCM_JLCPCB:C_0805, symbol PCM_JLCPCB-Capacitors:0805,100nF
- added C7: 1uF, PCM_JLCPCB:C_0805, symbol PCM_JLCPCB-Capacitors:0805,1uF
- added H1, H2, H3, H4: MountingHole, MountingHole:MountingHole_3.2mm_M3, symbol Mechanical:MountingHole
- added TP1, TP2, TP3: TestPoint, TestPoint:TestPoint_Pad_D1.5mm, symbol Connector:TestPoint
- C1: renamed from C2; value 1u -> 1uF; footprint Capacitor_SMD:C_0805_2012Metric -> PCM_JLCPCB:C_0805
- C2: renamed from C1; footprint PCM_JLCPCB:C_0603 -> PCM_JLCPCB:C_0805; JLCPCB (none) -> C28233
- C3: renamed from C4; value 1u -> 1uF; footprint Capacitor_SMD:C_0805_2012Metric -> PCM_JLCPCB:C_0805
- C4: renamed from C3; footprint PCM_JLCPCB:C_0603 -> PCM_JLCPCB:C_0805; JLCPCB (none) -> C28233
- D1: renamed from D2; footprint Diode_SMD:D_0201_0603Metric -> PCM_JLCPCB:D_0603
- JP1: renamed from JP4; footprint (none) -> Connector_PinHeader_2.54mm:PinHeader_1x02_P2.54mm_Vertical; now left out of the parts list
- JP2: renamed from JP5; footprint (none) -> Connector_PinHeader_2.54mm:PinHeader_1x02_P2.54mm_Vertical; now left out of the parts list
- Q1: renamed from Q2; value SS8050 -> L8050QLT1G; LCSC C7420370 -> C49581; Part SS8050 -> L8050QLT1G; now left out of the parts list
- Q2: renamed from Q3; value SS8050 -> L8050QLT1G; now left out of the parts list
- R1: renamed from R8; JLCPCB (none) -> C116677; now left out of the parts list
- R2: renamed from R13; JLCPCB (none) -> C116677; now left out of the parts list
- R3: footprint Resistor_SMD:R_0805_2012Metric -> PCM_JLCPCB:R_0603; JLCPCB C17513 -> C22548; now left out of the parts list
- R6: renamed from R38; JLCPCB (none) -> C99782; now left out of the parts list
- R7: renamed from R9; JLCPCB (none) -> C116677; now left out of the parts list
- R8: renamed from R42; JLCPCB (none) -> C99782; now left out of the parts list
- S1: footprint PCM_JLCPCB:SW-SMD_4P-L5.1-W5.1-P3.70-LS6.5-TL-2 -> (none); JLCPCB (none) -> C720477; LCSC C318884 -> C720477; Part TS-1187A-B-A-B -> TS-1088-AR02016; now left out of the parts list
- S2: footprint PCM_JLCPCB:SW-SMD_4P-L5.1-W5.1-P3.70-LS6.5-TL-2 -> (none); JLCPCB (none) -> C720477; now left out of the parts list
- U2: renamed from U4; footprint (none) -> PCM_Espressif:ESP32-S3-WROOM-1
- renumbered R10 to R4, R12 to R5
Connections:
- net ESP_3V3 is gone; now on net +3V3: R7.2, U2.2 (3V3)
- net +3V3: now also C15.1, C6.1, TP3.1; no longer C1.1, C2.2, C3.2, C4.2, R3.2, S1.1 (A), S2.1 (A), U1.1 (GND), U2.1 (GND)
- net +5V: now also TP1.1
- net CHIP_PU: now also C7.1
- net USB_DN-ESP renamed USB_ESP-DN
- net USB_DP-ESP renamed USB_ESP-DP
- new net GND: C1.1, C15.2, C2.2, C3.2, C4.2, C6.2, C7.2, R3.2, S1.1 (A), S2.1 (A), TP2.1, U1.1 (GND), U2.1 (GND)

Commit message: new footprints complete
Parts:
- C15: JLCPCB C237493 -> C15850
- C6: JLCPCB C49678 -> C28233
- D1: footprint PCM_JLCPCB:D_0603 -> PCM_JLCPCB:D_0805; JLCPCB C2286 -> C84256; now left out of the parts list
- Q1: footprint PCM_JLCPCB:Q_SOT-23 -> PCM_JLCPCB:D_SOT-23
- Q2: footprint PCM_JLCPCB:Q_SOT-23 -> PCM_JLCPCB:D_SOT-23; LCSC C7420370 -> C49581
- R1, R2, R7: LCSC C25804 -> C116677
- R6, R8: LCSC C23162 -> C99782
- S1, S2: footprint (none) -> PCM_JLCPCB:SW_TS-1088-AR02016
- TP2: footprint TestPoint:TestPoint_Pad_D1.5mm -> TestPoint:TestPoint_Pad_1.5x1.5mm
Changed lines of the file:
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@@
 			)
 		)
-		(property "Footprint" "PCM_JLCPCB:Q_SOT-23"
+		(property "Footprint" "PCM_JLCPCB:D_SOT-23"
 			(at 62.992 95.25 90)
 			(hide yes)
@@
 			)
 		)
-		(property "LCSC" "C7420370"
+		(property "LCSC" "C49581"
 			(at 64.77 95.25 0)
 			(hide yes)
@@
 			)
 		)
-		(property "LCSC" "C25804"
+		(property "LCSC" "C116677"
 			(at 142.24 59.69 0)
 			(hide yes)
@@
 			)
 		)
-		(property "LCSC" "C25804"
+		(property "LCSC" "C116677"
 			(at 53.34 78.74 0)
 			(hide yes)
@@
 			)
 		)
-		(property "JLCPCB" "C237493"
+		(property "JLCPCB" "C15850"
 			(at 162.56 40.64 0)
 			(hide yes)
@@
 			)
 		)
-		(property "Footprint" "PCM_JLCPCB:Q_SOT-23"
+		(property "Footprint" "PCM_JLCPCB:D_SOT-23"
 			(at 62.992 78.74 90)
 			(hide yes)
@@
 			)
 		)
-		(property "LCSC" "C23162"
+		(property "LCSC" "C99782"
 			(at 142.24 163.83 0)
 			(hide yes)
@@
 		(body_style 1)
 		(exclude_from_sim no)
-		(in_bom yes)
+		(in_bom no)
 		(on_board yes)
 		(in_pos_files yes)
@@
 			)
 		)
-		(property "Footprint" "PCM_JLCPCB:D_0603"
+		(property "Footprint" "PCM_JLCPCB:D_0805"
 			(at 63.5 31.75 0)
 			(hide yes)
@@
 			)
 		)
-		(property "JLCPCB" "C2286"
+		(property "JLCPCB" "C84256"
 			(at 63.5 31.75 0)
 			(hide yes)
@@
 			)
 		)
-		(property "LCSC" "C25804"
+		(property "LCSC" "C116677"
 			(at 53.34 95.25 0)
 			(hide yes)
@@
 			)
 		)
-		(property "JLCPCB" "C49678"
+		(property "JLCPCB" "C28233"
 			(at 167.64 40.64 0)
 			(hide yes)
@@
 			)
 		)
-		(property "Footprint" "TestPoint:TestPoint_Pad_D1.5mm"
+		(property "Footprint" "TestPoint:TestPoint_Pad_1.5x1.5mm"
 			(at 59.69 50.8 0)
 			(hide yes)
@@
 			)
 		)
-		(property "LCSC" "C23162"
+		(property "LCSC" "C99782"
 			(at 132.08 163.83 0)
 			(hide yes)
@@
 			)
 		)
-		(property "Footprint" ""
+		(property "Footprint" "PCM_JLCPCB:SW_TS-1088-AR02016"
 			(at 83.82 138.43 0)
 			(hide yes)
@@
 			)
 		)
-		(property "Footprint" ""
+		(property "Footprint" "PCM_JLCPCB:SW_TS-1088-AR02016"
 			(at 40.64 139.7 0)
 			(hide yes)
