File: dualpress/display.kicad_sch (KiCad schematic)
At the start: 1 part, among them U2 2.8" Touch Display SPI 14x1

Commit message: schematic done
Parts:
- removed U2: 2.8" Touch Display SPI 14x1, Connector_PinHeader_2.54mm:PinHeader_1x14_P2.54mm_Vertical, symbol 01_dualpress:2.8{dblquote} Touch Display SPI 14x1
