File: dualpress/dualpress.kicad_pcb (KiCad board)
At the start: 2 copper layers, 86 x 50 mm, 17 parts, among them J1 WATCH_RELAIS, J2 CTRL_RELAIS, J3 WATCH_PRESSURE, J4 WATCH_VALVE, U1 ESP32-S3-DEVKITC-1-N8R2, U2 2.8" Touch Display SPI 14x1, U3 PC817, U5 AMS1117

Commit message: schematic done
Parts:
- removed C1, C4: 10u, Capacitor_Tantalum_SMD:CP_EIA-3528-21_Kemet-B_HandSolder
- removed C2, C3: 1u, Capacitor_SMD:C_0805_2012Metric
- removed D1, D2: LED, Diode_SMD:D_0201_0603Metric
- removed J1: WATCH_RELAIS, Connector_JST:JST_XH_B2B-XH-AM_1x02_P2.50mm_Vertical
- removed J2: CTRL_RELAIS, Connector_JST:JST_XH_B2B-XH-AM_1x02_P2.50mm_Vertical
- removed J3: WATCH_PRESSURE, Connector_JST:JST_XH_B2B-XH-AM_1x02_P2.50mm_Vertical
- removed J4: WATCH_VALVE, Connector_JST:JST_XH_B2B-XH-AM_1x02_P2.50mm_Vertical
- removed JP1: Jumper_2_Open, Connector_PinHeader_2.54mm:PinHeader_1x02_P2.54mm_Vertical
- removed R1: 470, Resistor_SMD:R_0805_2012Metric
- removed R3: 1k, Resistor_SMD:R_0805_2012Metric
- removed U1: ESP32-S3-DEVKITC-1-N8R2, 01_dualpress:XCVR_ESP32-S3-DEVKITC-1-N8R2
- removed U2: 2.8" Touch Display SPI 14x1, Connector_PinHeader_2.54mm:PinHeader_1x14_P2.54mm_Vertical
- removed U3: PC817, Package_DIP:DIP-4_W7.62mm
- removed U5: AMS1117, PCM_JLCPCB:SOT-223-3_L6.5-W3.4-P2.30-LS7.0-BR
Routing:
- net /GPIO_4: track 74.2 -> 0.00 mm, vias 4 -> 0
- net /GPIO_6: track 71.7 -> 0.00 mm, vias 5 -> 0
- net /GPIO_5: track 71.1 -> 0.00 mm
- net /GPIO_15: track 63.1 -> 0.00 mm, vias 2 -> 0
- net /GPIO_11: track 57.5 -> 0.00 mm, vias 2 -> 0
- net /GPIO_7: track 55.2 -> 0.00 mm, vias 2 -> 0
- net /GPIO_8: track 52.0 -> 0.00 mm, vias 2 -> 0
- net /GPIO_10: track 51.9 -> 0.00 mm, vias 2 -> 0
- net /GPIO_9: track 46.7 -> 0.00 mm
- net /GPIO_12: track 43.8 -> 0.00 mm, vias 2 -> 0
- net /GPIO_13: track 38.7 -> 0.00 mm, vias 1 -> 0
- net Net-(D2-A): track 20.3 -> 0.00 mm
- net +3V3: track 13.8 -> 0.00 mm
- net GND: track 10.2 -> 0.00 mm, vias 6 -> 0
- net Net-(JP1-A): track 9.58 -> 0.00 mm
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- removed copper zone on B.Cu, net GND
Other:
- board outline removed
- copper layers 2 -> 4

Commit message: before remove footprints
Parts:
- added C1: 1uF, PCM_JLCPCB:C_0805, F.Cu at (139.2, 121.2)
- added C11: 100nF, PCM_JLCPCB:C_0805, F.Cu at (-31.3, 172.7)
- added C12: 1uF, PCM_JLCPCB:C_0805, F.Cu at (-31.3, 177.7)
- added C15: 10uF, PCM_JLCPCB:C_0805, F.Cu at (-37.7, 172.7)
- added C16: 10uF, PCM_JLCPCB:C_0805, F.Cu at (-37.7, 177.7)
- added C17: 10uF, PCM_JLCPCB:C_0805, F.Cu at (-37.7, 180.8)
- added C18: 10uF, PCM_JLCPCB:C_0805, F.Cu at (-31.3, 180.8)
- added C2: 100nF, PCM_JLCPCB:C_0805, F.Cu at (121.8, 101.2)
- added C3: 1uF, PCM_JLCPCB:C_0805, F.Cu at (139.2, 124.2)
- added C4: 100nF, PCM_JLCPCB:C_0805, F.Cu at (122.5, 119.4)
- added C6: 100nF, PCM_JLCPCB:C_0805, F.Cu at (-37.7, 166.6)
- added C7: 1uF, PCM_JLCPCB:C_0805, F.Cu at (-37.7, 169.6)
- added C8: 100nF, PCM_JLCPCB:C_0805, F.Cu at (-31.3, 166.6)
- added C9: 100nF, PCM_JLCPCB:C_0805, F.Cu at (-31.3, 169.6)
- added D1: LED, PCM_JLCPCB:D_0603, F.Cu at (145.2, 116.7)
- added D2: SMBJ6.5CA, PCM_JLCPCB:D_SMB, F.Cu at (193.8, 97.6)
- added D3: SMBJ6.5CA, PCM_JLCPCB:D_SMB, F.Cu at (122.7, 112.7)
- added D4: SMBJ6.5CA, PCM_JLCPCB:D_SMB, F.Cu at (188.8, 97.8)
- added D5: SMBJ6.5CA, PCM_JLCPCB:D_SMB, F.Cu at (130.6, 104.6)
- added D6: 1N5819HW-7-F, PCM_JLCPCB:D_SOD-123, F.Cu at (194.6, 103.8)
- added D7: 1N5819HW-7-F, PCM_JLCPCB:D_SOD-123, F.Cu at (121.8, 105.0)
- added D8: SMBJ6.5CA, PCM_JLCPCB:D_SMB, F.Cu at (183.6, 97.8)
- added D9: SMBJ6.5CA, PCM_JLCPCB:D_SMB, F.Cu at (130.6, 115.7)
- added H1: MountingHole, MountingHole:MountingHole_3.2mm_M3, F.Cu at (201.7, 89.6)
- added H2: MountingHole, MountingHole:MountingHole_3.2mm_M3, F.Cu at (201.5, 150.4)
- added H3: MountingHole, MountingHole:MountingHole_3.2mm_M3, F.Cu at (109.5, 89.4)
- added H4: MountingHole, MountingHole:MountingHole_3.2mm_M3, F.Cu at (110.7, 150.0)
- added J1: Connector, USB-TYPE-C-16P, PCM_JLCPCB:TYPE-C-SMD_HX-TYPE-C-16PIN, F.Cu at (188.1, 89.2)
- added J10: Conn_01x06_Pin, Connector_JST:JST_XH_B6B-XH-AM_1x06_P2.50mm_Vertical, F.Cu at (71.0, 150.0)
- added J2: Connector, USB-TYPE-C-16P, PCM_JLCPCB:TYPE-C-SMD_HX-TYPE-C-16PIN, F.Cu at (115.8, 107.4)
- added J3: TC2030, Connector:Tag-Connect_TC2030-IDC-NL_2x03_P1.27mm_Vertical, F.Cu at (121.8, 126.0)
- added J4: VALVE, TerminalBlock:TerminalBlock_MaiXu_MX126-5.0-02P_1x02_P5.00mm, F.Cu at (201.8, 134.4)
- added J5: RELAIS, TerminalBlock:TerminalBlock_MaiXu_MX126-5.0-02P_1x02_P5.00mm, F.Cu at (201.8, 120.7)
- added J6: PRESSURE, TerminalBlock:TerminalBlock_MaiXu_MX126-5.0-03P_1x03_P5.00mm, F.Cu at (149.6, 148.7)
- added J7: SSR CTRL, TerminalBlock:TerminalBlock_MaiXu_MX126-5.0-02P_1x02_P5.00mm, F.Cu at (126.2, 149.5)
- added J8: Conn_01x06_Pin, Connector_JST:JST_XH_B6B-XH-AM_1x06_P2.50mm_Vertical, F.Cu at (118.1, 88.8)
- added J9: Conn_01x06_Pin, Connector_JST:JST_XH_B6B-XH-AM_1x06_P2.50mm_Vertical, F.Cu at (154.5, 120.2)
- added JP1: Jumper_2_Open, Connector_PinHeader_2.54mm:PinHeader_1x02_P2.54mm_Vertical, F.Cu at (165.9, 92.3)
- added JP2: Jumper_2_Open, Connector_PinHeader_2.54mm:PinHeader_1x02_P2.54mm_Vertical, F.Cu at (170.5, 92.3)
- added JP3: Jumper_3_Open, Connector_PinHeader_2.54mm:PinHeader_1x03_P2.54mm_Vertical, F.Cu at (121.4, 142.6)
- added JP4: Jumper_3_Open, Connector_PinHeader_2.54mm:PinHeader_1x03_P2.54mm_Vertical, F.Cu at (121.2, 133.8)
- added JP5: Jumper_3_Open, Connector_PinHeader_2.54mm:PinHeader_1x03_P2.54mm_Vertical, F.Cu at (121.2, 138.3)
- added Q1: L8050QLT1G, PCM_JLCPCB:Q_SOT-23, F.Cu at (148.3, 109.1)
- added Q2: L8050QLT1G, PCM_JLCPCB:Q_SOT-23, F.Cu at (152.9, 109.1)
- added Q3: L8050QLT1G, PCM_JLCPCB:Q_SOT-23, F.Cu at (119.3, 149.2)
- added Q4: AO3401A, Package_TO_SOT_SMD:SOT-23, F.Cu at (175.3, 146.3)
- added R1: 10kΩ, PCM_JLCPCB:R_0603, F.Cu at (147.0, 113.3)
- added R10: 5.1kΩ, PCM_JLCPCB:R_0603, F.Cu at (136.6, 109.8)
- added R11: 5.1kΩ, PCM_JLCPCB:R_0603, F.Cu at (190.1, 103.4)
- added R12: 5.1kΩ, PCM_JLCPCB:R_0603, F.Cu at (136.6, 112.0)
- added R13: 220kΩ, PCM_JLCPCB:R_0603, F.Cu at (167.8, 100.6)
- added R14: 47kΩ, PCM_JLCPCB:R_0603, F.Cu at (170.0, 100.6)
- added R15: 1kΩ, PCM_JLCPCB:R_0603, F.Cu at (165.5, 100.6)
- added R16: 10k (1%), PCM_JLCPCB:R_0603, F.Cu at (166.7, 112.4)
- added R2: 10kΩ, PCM_JLCPCB:R_0603, F.Cu at (156.0, 113.3)
- added R22: 300k, Capacitor_THT:CP_Axial_L11.0mm_D5.0mm_P18.00mm_Horizontal, F.Cu at (176.8, 121.9)
- added R23: 47kΩ, PCM_JLCPCB:R_0603, F.Cu at (160.8, 134.4)
- added R24: 47kΩ, PCM_JLCPCB:R_0603, F.Cu at (161.2, 122.6)
- added R25: 1kΩ, PCM_JLCPCB:R_0603, F.Cu at (144.7, 139.1)
- added R26: 15kΩ, PCM_JLCPCB:R_0603, F.Cu at (146.8, 141.8)
- added R27: 10kΩ, PCM_JLCPCB:R_0603, F.Cu at (148.7, 139.1)
- added R28: 0Ω, PCM_JLCPCB:R_0603, F.Cu at (133.3, 98.3)
- added R29: 1kΩ, PCM_JLCPCB:R_0603, F.Cu at (119.0, 152.3)
- added R3: 1k, PCM_JLCPCB:R_0603, F.Cu at (138.8, 127.9)
- added R30: 330Ω, PCM_JLCPCB:R_0603, F.Cu at (133.3, 96.0)
- added R31: 100Ω, PCM_JLCPCB:R_0805, F.Cu at (167.1, 146.6)
- added R32: 100kΩ, PCM_JLCPCB:R_0603, F.Cu at (170.1, 146.6)
- added R33: 10kΩ, PCM_JLCPCB:R_0603, F.Cu at (132.8, 140.1)
- added R34: 0Ω, PCM_JLCPCB:R_0603, F.Cu at (133.4, 136.1)
- added R35: 0Ω, PCM_JLCPCB:R_0603, F.Cu at (133.0, 131.4)
- added R36: 10kΩ, PCM_JLCPCB:R_0603, F.Cu at (130.6, 140.1)
- added R37: 10kΩ, PCM_JLCPCB:R_0603, F.Cu at (135.0, 140.1)
- added R38: 0Ω, PCM_JLCPCB:R_0603, F.Cu at (133.0, 133.7)
- added R39: 300Ω, PCM_JLCPCB:R_1206, F.Cu at (156.2, 142.0)
- added R4: 0Ω, PCM_JLCPCB:R_0603, F.Cu at (151.5, 113.3)
- added R40: 300Ω, PCM_JLCPCB:R_1206, F.Cu at (156.2, 145.3)
- added R41: 300Ω, PCM_JLCPCB:R_1206, F.Cu at (154.6, 137.9)
- added R42: 300k, Capacitor_THT:CP_Axial_L11.0mm_D5.0mm_P18.00mm_Horizontal, F.Cu at (176.9, 133.9)
- added R5: 0Ω, PCM_JLCPCB:R_0603, F.Cu at (153.8, 113.3)
- added R6: 4.7kΩ, PCM_JLCPCB:R_0603, F.Cu at (165.4, 86.7)
- added R7: 10kΩ, PCM_JLCPCB:R_0603, F.Cu at (136.7, 88.9)
- added R8: 4.7kΩ, PCM_JLCPCB:R_0603, F.Cu at (165.4, 88.9)
- added R9: 5.1kΩ, PCM_JLCPCB:R_0603, F.Cu at (192.3, 103.4)
- added S1: Tactile Button, 160gf, PCM_JLCPCB:SW-SMD_4P-L5.1-W5.1-P3.70-LS6.5-TL-2, F.Cu at (115.9, 97.1)
- added S2: Tactile Button, 160gf, PCM_JLCPCB:SW-SMD_4P-L5.1-W5.1-P3.70-LS6.5-TL-2, F.Cu at (115.7, 117.5)
- added TP1: TestPoint, TestPoint:TestPoint_Pad_D1.5mm, F.Cu at (143.2, 125.0)
- added TP10: TestPoint, TestPoint:TestPoint_Pad_D1.5mm, F.Cu at (148.0, 136.0)
- added TP2: TestPoint, TestPoint:TestPoint_Pad_D1.5mm, F.Cu at (143.2, 128.5)
- added TP3: TestPoint, TestPoint:TestPoint_Pad_D1.5mm, F.Cu at (143.2, 121.4)
- added TP4: TestPoint, TestPoint:TestPoint_Pad_D1.5mm, F.Cu at (164.7, 139.7)
- added TP5: TestPoint, TestPoint:TestPoint_Pad_D1.5mm, F.Cu at (164.2, 126.4)
- added TP6: TestPoint, TestPoint:TestPoint_Pad_D1.5mm, F.Cu at (162.0, 137.5)
- added TP7: TestPoint, TestPoint:TestPoint_Pad_D1.5mm, F.Cu at (161.2, 126.4)
- added TP8: TestPoint, TestPoint:TestPoint_Pad_D1.5mm, F.Cu at (141.0, 136.0)
- added TP9: TestPoint, TestPoint:TestPoint_Pad_D1.5mm, F.Cu at (144.5, 136.0)
- added U1: LD1117S33TR_SOT223, Package_TO_SOT_SMD:SOT-223-3_TabPin2, F.Cu at (132.1, 123.8)
- added U2: ~, PCM_Espressif:ESP32-S3-WROOM-1, F.Cu at (151.8, 95.1)
- added U3: CP2102N-Axx-xQFN28, Package_DFN_QFN:QFN-28-1EP_5x5mm_P0.5mm_EP3.35x3.35mm, F.Cu at (168.3, 106.3)
- added U4: LTV-814, Package_DIP:DIP-4_W7.62mm, F.Cu at (172.4, 132.6)
- added U5: LTV-814, Package_DIP:DIP-4_W7.62mm, F.Cu at (172.4, 121.6)
- added U6: 2.8" Touch Display SPI 14x1, Connector_PinHeader_2.54mm:PinHeader_1x14_P2.54mm_Vertical, F.Cu at (189.7, 150.9)
- added U7: SSR-41FDD, 01_dualpress:SSR-41FDD, F.Cu at (178.9, 142.5)
Other:
- board outline added: 100.8 x 70.4 mm
