File: dualpress/sensors.kicad_sch (KiCad schematic)
At the start: 5 parts, among them J1 WATCH_RELAIS, U3 PC817

Commit message: schematic done
Parts:
- removed D1: LED, Diode_SMD:D_0201_0603Metric, symbol Device:LED
- removed R1: 470, Resistor_SMD:R_0805_2012Metric, symbol Device:R
- removed R2: R, symbol Device:R
- removed U3: PC817, Package_DIP:DIP-4_W7.62mm, symbol Isolator:PC817
- added C12, C13, C14: 100nF, PCM_JLCPCB:C_0603, symbol PCM_JLCPCB-Capacitors:0603,100nF
- added J2: VALVE, Connector_JST:JST_XH_B2B-XH-AM_1x02_P2.50mm_Vertical, symbol Connector:Screw_Terminal_01x02
- added J6: PRESSURE, symbol Connector:Screw_Terminal_01x03
- added R1, R2: 47kΩ, PCM_JLCPCB:R_0603, symbol PCM_JLCPCB-Resistors:0603,47kΩ
- added R26: 10kΩ, PCM_JLCPCB:R_0603, symbol PCM_JLCPCB-Resistors:0603,10kΩ
- added R29: 1kΩ, PCM_JLCPCB:R_0603, symbol PCM_JLCPCB-Resistors:0603,1kΩ
- added R30: 15kΩ, PCM_JLCPCB:R_0603, symbol PCM_JLCPCB-Resistors:0603,15kΩ
- added R32, R33, R34, R35, R36, R37: 100k, Plugin,D4.5xL11.5mm, symbol Device:R
- added U3, U6: LTV-814, Package_DIP:DIP-4_W7.62mm, symbol Isolator:LTV-814
- J1: value WATCH_RELAIS -> RELAIS
Connections:
- net +5V: now also J6.1 (Pin_1)
- net GND: now also C12.2, C13.2, C14.2, J6.3 (Pin_3), R30.2, U3.3, U6.3
- net at J1.1 (Pin_1): now also R32.1
- net at J1.2 (Pin_2): now also U3.2
- new net: R26.1, R29.2, R30.1
- new net: J6.2 (Pin_2), R26.2
- new net: R35.2, R36.1
- new net: R36.2, R37.1
- new net: J2.1 (Pin_1), R35.1
- new net: R34.2, U3.1
- new net: R37.2, U6.1
- new net: J2.2 (Pin_2), U6.2
- new net: R32.2, R33.1
- new net: R33.2, R34.1
- new net +3V3: R1.1, R2.1
- new net SENS_PRESSURE: C12.1, R29.1
- new net SENS_RELAY: C13.1, R1.2, U3.4
- new net SENS_VALVE: C14.1, R2.2, U6.4
Other:
- note added: "PRESSURE"
- note added: "RELAIS"
- note added: "VALVE"
- moved on the sheet: J1

Commit message: before remove footprints
Parts:
- removed C12, C13, C14: 100nF, PCM_JLCPCB:C_0603, symbol PCM_JLCPCB-Capacitors:0603,100nF
- removed R32, R33, R34, R35, R36, R37: 100k, Plugin,D4.5xL11.5mm, symbol Device:R
- added C11, C8, C9: 100nF, PCM_JLCPCB:C_0805, symbol PCM_JLCPCB-Capacitors:0805,100nF
- added R22, R42: 300k, Capacitor_THT:CP_Axial_L11.0mm_D5.0mm_P18.00mm_Horizontal, symbol Device:R
- added TP10, TP4, TP5, TP6, TP7, TP8, TP9: TestPoint, TestPoint:TestPoint_Pad_D1.5mm, symbol Connector:TestPoint
- J4: renamed from J2; footprint Connector_JST:JST_XH_B2B-XH-AM_1x02_P2.50mm_Vertical -> TerminalBlock:TerminalBlock_MaiXu_MX126-5.0-02P_1x02_P5.00mm; now left out of the parts list
- J5: renamed from J1; footprint Connector_JST:JST_XH_B2B-XH-AM_1x02_P2.50mm_Vertical -> TerminalBlock:TerminalBlock_MaiXu_MX126-5.0-02P_1x02_P5.00mm; now left out of the parts list
- J6: footprint (none) -> TerminalBlock:TerminalBlock_MaiXu_MX126-5.0-03P_1x03_P5.00mm; now left out of the parts list
- R25: renamed from R29; JLCPCB (none) -> C22548; now left out of the parts list
- R27: renamed from R26; JLCPCB (none) -> C116677; now left out of the parts list
- renumbered R2 to R23, R1 to R24, R30 to R26, U6 to U4, U3 to U5
Connections:
- net GND: now also C11.2, C8.2, C9.2, TP10.1, TP6.1, TP7.1
- net SENS_PRESSURE: now also C11.1
- net SENS_RELAY: now also C8.1, TP5.1
- net SENS_VALVE: now also C9.1, TP4.1
- net at R25.2, R26.1, R27.1: now also TP8.1
- net at J6.2 (Pin_2), R27.2: now also TP9.1
- net at J4.1 (Pin_1): now also R42.2
- net at U5.1: now also R22.1
- net at U4.1: now also R42.1
- net at J5.1 (Pin_1): now also R22.2
Other:
- note added: "AC"
- moved on the sheet: J4, J5

Commit message: new footprints complete
Parts:
- removed R42: 300k, Capacitor_THT:CP_Axial_L11.0mm_D5.0mm_P18.00mm_Horizontal, symbol Device:R
- removed U4, U5: LTV-814, Package_DIP:DIP-4_W7.62mm, symbol Isolator:LTV-814
- added R43: 300k, Resistor_THT:R_Axial_DIN0414_L11.9mm_D4.5mm_P15.24mm_Horizontal, symbol Device:R
- added U8, U9: SFH620A-3X001, Package_DIP:DIP-4_W7.62mm, symbol Isolator:SFH620A-3X001
- C11, C8, C9: JLCPCB C49678 -> C28233
- J4, J5: footprint TerminalBlock:TerminalBlock_MaiXu_MX126-5.0-02P_1x02_P5.00mm -> 01_dualpress:KF2EDGV-3.5-2P
- J6: footprint TerminalBlock:TerminalBlock_MaiXu_MX126-5.0-03P_1x03_P5.00mm -> 01_dualpress:KF2EDGV-3.5-3P
- R22: footprint Capacitor_THT:CP_Axial_L11.0mm_D5.0mm_P18.00mm_Horizontal -> Resistor_THT:R_Axial_DIN0414_L11.9mm_D4.5mm_P15.24mm_Horizontal; now fitted
- R25: LCSC C21190 -> C22548
- R27: LCSC C25804 -> C116677
- TP10, TP6, TP7: footprint TestPoint:TestPoint_Pad_D1.5mm -> TestPoint:TestPoint_Pad_1.5x1.5mm
Connections:
- net GND: now also U8.3, U9.3
- net SENS_RELAY: now also U9.4
- net SENS_VALVE: now also U8.4
- net at R22.1: now also U9.1
- net at J5.2 (Pin_2): now also U9.2
- net at J4.2 (Pin_2): now also U8.2
- net at J4.1 (Pin_1): now also R43.2
- new net: R43.1, U8.1
Changed lines of the file:
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@@
 	)
 	(symbol
+		(lib_id "Isolator:SFH620A-3X001")
+		(at 107.95 74.93 0)
+		(unit 1)
+		(body_style 1)
+		(exclude_from_sim no)
+		(in_bom no)
+		(on_board yes)
+		(in_pos_files yes)
+		(dnp no)
+		(fields_autoplaced yes)
+		(property "Reference" "U9"
+			(at 107.95 64.77 0)
+			(show_name no)
+			(do_not_autoplace no)
+			(effects
+				(font
+					(size 1.27 1.27)
+				)
+			)
+		)
+		(property "Value" "SFH620A-3X001"
+			(at 107.95 67.31 0)
+			(show_name no)
+			(do_not_autoplace no)
+			(effects
+				(font
+					(size 1.27 1.27)
+				)
+			)
+		)
+		(property "Footprint" "Package_DIP:DIP-4_W7.62mm"
+			(at 107.95 85.09 0)
+			(hide yes)
+			(show_name no)
+			(do_not_autoplace no)
+			(effects
+				(font
+					(size 1.27 1.27)
+				)
+			)
+		)
+		(property "Datasheet" "http://www.vishay.com/docs/83675/sfh620a.pdf"
+			(at 106.68 74.93 0)
+			(hide yes)
+			(show_name no)
+			(do_not_autoplace no)
+			(effects
+				(font
+					(size 1.27 1.27)
+				)
+			)
+		)
+		(property "Description" "Optocoupler, Phototransistor Output, 5300 VRMS, VCEO 70V, CTR% 100-320 VDE, UL, CUL, BSI, THT PDIP-4"
+			(at 107.95 74.93 0)
+			(hide yes)
+			(show_name no)
+			(do_not_autoplace no)
+			(effects
+				(font
+					(size 1.27 1.27)
+				)
+			)
+		)
+		(pin "3"
+		)
+		(pin "1"
+		)
+		(pin "2"
+		)
+		(pin "4"
+		)
+		(instances
+			(project "dualpress"
+				(path "/4c49edca-ce86-4659-a271-9f68536bc424/543aee8e-2b2f-4977-9416-02d65e4a96d7"
+					(reference "U9")
+					(unit 1)
+				)
+			)
+		)
+	)
+	(symbol
 		(lib_id "Connector:TestPoint")
 		(at 134.62 82.55 0)
@@
 			)
 		)
-		(property "Footprint" "TestPoint:TestPoint_Pad_D1.5mm"
+		(property "Footprint" "TestPoint:TestPoint_Pad_1.5x1.5mm"
 			(at 139.7 82.55 0)
 			(hide yes)
@@
 			)
 		)
-		(property "LCSC" "C25804"
+		(property "LCSC" "C116677"
 			(at 220.98 92.71 0)
 			(hide yes)
@@
 			)
 		)
-		(property "JLCPCB" "C49678"
+		(property "JLCPCB" "C28233"
 			(at 201.93 100.33 0)
 			(hide yes)
@@
 	)
 	(symbol
-		(lib_id "Isolator:LTV-814")
-		(at 107.95 74.93 0)
+		(lib_id "Isolator:SFH620A-3X001")
+		(at 105.41 147.32 0)
 		(unit 1)
 		(body_style 1)
 		(exclude_from_sim no)
-		(in_bom yes)
+		(in_bom no)
 		(on_board yes)
 		(in_pos_files yes)
 		(dnp no)
 		(fields_autoplaced yes)
-		(property "Reference" "U5"
-			(at 107.95 66.04 0)
+		(property "Reference" "U8"
+			(at 105.41 137.16 0)
 			(show_name no)
 			(do_not_autoplace no)
@@
 			)
 		)
-		(property "Value" "LTV-814"
-			(at 107.95 68.58 0)
+		(property "Value" "SFH620A-3X001"
+			(at 105.41 139.7 0)
 			(show_name no)
 			(do_not_autoplace no)
@@
 		)
 		(property "Footprint" "Package_DIP:DIP-4_W7.62mm"
-			(at 102.87 80.01 0)
+			(at 105.41 157.48 0)
 			(hide yes)
 			(show_name no)
@@
 				(font
 					(size 1.27 1.27)
-					(italic yes)
 				)
-				(justify left)
 			)
 		)
-		(property "Datasheet" "https://optoelectronics.liteon.com/upload/download/DS-70-96-0013/LTV-8X4%20series%20201509.pdf"
-			(at 109.855 74.93 0)
+		(property "Datasheet" "http://www.vishay.com/docs/83675/sfh620a.pdf"
+			(at 104.14 147.32 0)
 			(hide yes)
 			(show_name no)
@@
 					(size 1.27 1.27)
 				)
-				(justify left)
 			)
 		)
-		(property "Description" "AC/DC Optocoupler, Vce 35V, CTR 20%, DIP4"
-			(at 107.95 74.93 0)
-			(hide yes)
-			(show_name no)
-			(do_not_autoplace no)
-			(effects
-				(font
-					(size 1.27 1.27)
-				)
-			)
-		)
-		(property "JLC" "C125118"
-			(at 107.95 74.93 0)
+		(property "Description" "Optocoupler, Phototransistor Output, 5300 VRMS, VCEO 70V, CTR% 100-320 VDE, UL, CUL, BSI, THT PDIP-4"
+			(at 105.41 147.32 0)
 			(hide yes)
 			(show_name no)
@@
 			)
 		)
-		(pin "2"
+		(pin "3"
 		)
 		(pin "1"
 		)
-		(pin "3"
+		(pin "2"
 		)
 		(pin "4"
@@
 			(project "dualpress"
 				(path "/4c49edca-ce86-4659-a271-9f68536bc424/543aee8e-2b2f-4977-9416-02d65e4a96d7"
-					(reference "U5")
+					(reference "U8")
 					(unit 1)
 				)
@@
 			)
 		)
-		(property "Footprint" "TestPoint:TestPoint_Pad_D1.5mm"
+		(property "Footprint" "TestPoint:TestPoint_Pad_1.5x1.5mm"
 			(at 241.3 104.14 0)
 			(hide yes)
@@
 	)
 	(symbol
-		(lib_id "Isolator:LTV-814")
-		(at 105.41 147.32 0)
+		(lib_id "Device:R")
+		(at 83.82 140.97 270)
+		(mirror x)
 		(unit 1)
 		(body_style 1)
@@
 		(in_pos_files yes)
 		(dnp no)
-		(fields_autoplaced yes)
-		(property "Reference" "U4"
-			(at 105.41 138.43 0)
+		(property "Reference" "R43"
+			(at 83.82 137.16 90)
 			(show_name no)
 			(do_not_autoplace no)
@@
 			)
 		)
-		(property "Value" "LTV-814"
-			(at 105.41 140.97 0)
+		(property "Value" "300k"
+			(at 83.82 134.62 90)
 			(show_name no)
 			(do_not_autoplace no)
@@
 			)
 		)
-		(property "Footprint" "Package_DIP:DIP-4_W7.62mm"
-			(at 100.33 152.4 0)
+		(property "Footprint" "Resistor_THT:R_Axial_DIN0414_L11.9mm_D4.5mm_P15.24mm_Horizontal"
+			(at 83.82 142.748 90)
 			(hide yes)
 			(show_name no)
@@
 				(font
 					(size 1.27 1.27)
-					(italic yes)
 				)
-				(justify left)
 			)
 		)
-		(property "Datasheet" "https://optoelectronics.liteon.com/upload/download/DS-70-96-0013/LTV-8X4%20series%20201509.pdf"
-			(at 107.315 147.32 0)
+		(property "Datasheet" ""
+			(at 83.82 140.97 0)
 			(hide yes)
 			(show_name no)
@@
 					(size 1.27 1.27)
 				)
-				(justify left)
 			)
 		)
-		(property "Description" "AC/DC Optocoupler, Vce 35V, CTR 20%, DIP4"
-			(at 105.41 147.32 0)
+		(property "Description" "Resistor"
+			(at 83.82 140.97 0)
 			(hide yes)
 			(show_name no)
@@
 			)
 		)
-		(property "JLC" "C125118"
-			(at 105.41 147.32 0)
+		(property "JLCPCB" "C601006"
+			(at 83.82 140.97 90)
 			(hide yes)
 			(show_name no)
@@
 		(pin "1"
 		)
-		(pin "3"
-		)
-		(pin "4"
-		)
 		(instances
 			(project "dualpress"
 				(path "/4c49edca-ce86-4659-a271-9f68536bc424/543aee8e-2b2f-4977-9416-02d65e4a96d7"
-					(reference "U4")
+					(reference "R43")
 					(unit 1)
 				)
@@
 			)
 		)
-		(property "JLCPCB" "C49678"
+		(property "JLCPCB" "C28233"
 			(at 128.27 74.93 0)
 			(hide yes)
@@
 			)
 		)
-		(property "Footprint" "TerminalBlock:TerminalBlock_MaiXu_MX126-5.0-03P_1x03_P5.00mm"
+		(property "Footprint" "01_dualpress:KF2EDGV-3.5-3P"
 			(at 232.41 92.71 0)
 			(hide yes)
@@
 			)
 		)
-		(property "JLCPCB" "C49678"
+		(property "JLCPCB" "C28233"
 			(at 125.73 147.32 0)
 			(hide yes)
@@
 		(in_bom no)
 		(on_board yes)
-		(in_pos_files no)
+		(in_pos_files yes)
 		(dnp no)
 		(property "Reference" "J4"
@@
 			)
 		)
-		(property "Footprint" "TerminalBlock:TerminalBlock_MaiXu_MX126-5.0-02P_1x02_P5.00mm"
+		(property "Footprint" "01_dualpress:KF2EDGV-3.5-2P"
 			(at 69.85 144.78 0)
 			(hide yes)
@@
 			)
 		)
-		(property "LCSC" "C21190"
+		(property "LCSC" "C22548"
 			(at 207.01 92.71 0)
 			(hide yes)
@@
 			)
 		)
-		(property "Footprint" "TestPoint:TestPoint_Pad_D1.5mm"
+		(property "Footprint" "TestPoint:TestPoint_Pad_1.5x1.5mm"
 			(at 137.16 154.94 0)
 			(hide yes)
@@
 	)
 	(symbol
-		(lib_id "Device:R")
-		(at 83.82 140.97 270)
-		(mirror x)
-		(unit 1)
-		(body_style 1)
-		(exclude_from_sim no)
-		(in_bom yes)
-		(on_board yes)
-		(in_pos_files no)
-		(dnp yes)
-		(property "Reference" "R42"
-			(at 83.82 137.16 90)
-			(show_name no)
-			(do_not_autoplace no)
-			(effects
-				(font
-					(size 1.27 1.27)
-				)
-			)
-		)
-		(property "Value" "300k"
-			(at 83.82 134.62 90)
-			(show_name no)
-			(do_not_autoplace no)
-			(effects
-				(font
-					(size 1.27 1.27)
-				)
-			)
-		)
-		(property "Footprint" "Capacitor_THT:CP_Axial_L11.0mm_D5.0mm_P18.00mm_Horizontal"
-			(at 83.82 142.748 90)
-			(hide yes)
-			(show_name no)
-			(do_not_autoplace no)
-			(effects
-				(font
-					(size 1.27 1.27)
-				)
-			)
-		)
-		(property "Datasheet" ""
-			(at 83.82 140.97 0)
-			(hide yes)
-			(show_name no)
-			(do_not_autoplace no)
-			(effects
-				(font
-					(size 1.27 1.27)
-				)
-			)
-		)
-		(property "Description" "Resistor"
-			(at 83.82 140.97 0)
-			(hide yes)
-			(show_name no)
-			(do_not_autoplace no)
-			(effects
-				(font
-					(size 1.27 1.27)
-				)
-			)
-		)
-		(property "JLCPCB" "C601006"
-			(at 83.82 140.97 90)
-			(hide yes)
-			(show_name no)
-			(do_not_autoplace no)
-			(effects
-				(font
-					(size 1.27 1.27)
-				)
-			)
-		)
-		(pin "2"
-		)
-		(pin "1"
-		)
-		(instances
-			(project "dualpress"
-				(path "/4c49edca-ce86-4659-a271-9f68536bc424/543aee8e-2b2f-4977-9416-02d65e4a96d7"
-					(reference "R42")
-					(unit 1)
-				)
-			)
-		)
-	)
-	(symbol
 		(lib_id "Connector:Screw_Terminal_01x02")
 		(at 76.2 72.39 0)
@@
 		(in_bom no)
 		(on_board yes)
-		(in_pos_files no)
+		(in_pos_files yes)
 		(dnp no)
 		(property "Reference" "J5"
@@
 			)
 		)
-		(property "Footprint" "TerminalBlock:TerminalBlock_MaiXu_MX126-5.0-02P_1x02_P5.00mm"
+		(property "Footprint" "01_dualpress:KF2EDGV-3.5-2P"
 			(at 76.2 72.39 0)
 			(hide yes)
@@
 		(in_bom yes)
 		(on_board yes)
-		(in_pos_files no)
-		(dnp yes)
+		(in_pos_files yes)
+		(dnp no)
 		(property "Reference" "R22"
 			(at 90.17 64.77 90)
@@
 			)
 		)
-		(property "Footprint" "Capacitor_THT:CP_Axial_L11.0mm_D5.0mm_P18.00mm_Horizontal"
+		(property "Footprint" "Resistor_THT:R_Axial_DIN0414_L11.9mm_D4.5mm_P15.24mm_Horizontal"
 			(at 90.17 70.358 90)
 			(hide yes)
