File: dualpress/usb_serial.kicad_sch (KiCad schematic)
At the start: 19 parts, among them Q2 SS8050, Q3 SS8050, U5 CP2102N-Axx-xQFN28

Commit message: schematic done
Parts:
- removed C1, C3: 100nF, PCM_JLCPCB:C_0603, symbol PCM_JLCPCB-Capacitors:0603,100nF
- removed D3: WS2812B, PCM_JLCPCB:LED_WS2812B_PLCC4_5.0x5.0mm_P3.2mm, symbol PCM_JLCPCB-Extended:LED, WS2812B, 5050
- removed Q2, Q3: SS8050, PCM_JLCPCB:Q_SOT-23, symbol PCM_JLCPCB-Transistors:NPN,SS8050,(2)
- removed R10, R12, R14: 0Ω, PCM_JLCPCB:R_0603, symbol PCM_JLCPCB-Resistors:0603,0Ω
- removed R13, R8: 10kΩ, PCM_JLCPCB:R_0603, symbol PCM_JLCPCB-Resistors:0603,10kΩ
- removed S1, S2: Tactile Button, 160gf, PCM_JLCPCB:SW-SMD_4P-L5.1-W5.1-P3.70-LS6.5-TL-2, symbol PCM_JLCPCB-Connectors_Buttons:Tactile Button, 160gf, 12V, 50mA, 5.1mm
Connections:
- no-connect marks 18 -> 15
Other:
- note added: "SERIAL"
- moved on the sheet: C5, C6, R4, R5, R6, R7, U5

Commit message: before remove footprints
Parts:
- removed C5: 10uF, PCM_JLCPCB:C_0805, symbol PCM_JLCPCB-Capacitors:0805,10uF
- removed C6: 1u, Capacitor_SMD:C_0805_2012Metric, symbol Device:C
- added C12: 1uF, PCM_JLCPCB:C_0805, symbol PCM_JLCPCB-Capacitors:0805,1uF
- added C18: 10uF, PCM_JLCPCB:C_0805, symbol PCM_JLCPCB-Capacitors:0805,10uF
- added J3: TC2030, Connector:Tag-Connect_TC2030-IDC-NL_2x03_P1.27mm_Vertical, symbol Connector:TC2030
- R15: renamed from R5; JLCPCB (none) -> C22548; now left out of the parts list
- R16: renamed from R4; footprint (none) -> PCM_JLCPCB:R_0603; JLCPCB (none) -> C116677
- U3: renamed from U5; now left out of the parts list
- renumbered R6 to R13, R7 to R14
Connections:
- net +3V3: now also C18.1
- net GND: now also C12.2, C18.2
- net at R13.2, R14.1, U3.8 (VBUS): now also C12.1

Commit message: new footprints complete
Parts:
- C18: JLCPCB C237493 -> C15850
- J3: footprint Connector:Tag-Connect_TC2030-IDC-NL_2x03_P1.27mm_Vertical -> Connector:Tag-Connect_TC2030-IDC-FP_2x03_P1.27mm_Vertical
- R15: LCSC C21190 -> C22548
Changed lines of the file:
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@@
 			)
 		)
-		(property "LCSC" "C21190"
+		(property "LCSC" "C22548"
 			(at 111.76 58.42 0)
 			(hide yes)
@@
 			)
 		)
-		(property "JLCPCB" "C237493"
+		(property "JLCPCB" "C15850"
 			(at 105.41 55.88 0)
 			(hide yes)
@@
 			)
 		)
-		(property "Footprint" "Connector:Tag-Connect_TC2030-IDC-NL_2x03_P1.27mm_Vertical"
+		(property "Footprint" "Connector:Tag-Connect_TC2030-IDC-FP_2x03_P1.27mm_Vertical"
 			(at 218.44 54.61 0)
 			(hide yes)
